Commit message: init

File: src/rm_gimbal_description/urdf/rm_gimbal.urdf.xacro (robot description, xacro)
@@ -10,5 +10,6 @@
     <child link="shoot" />
   </joint>
-  <joint name="gimbal_joint" type="floating">
+  <joint name="gimbal_joint" type="fixed">
+    <origin xyz="0 0 0" rpy="0 0 0" />
     <parent link="odom" />
     <child link="gimbal_link" />

Commit message: init

File: src/rm_gimbal_description/urdf/rm_gimbal.urdf.xacro (robot description, xacro)
@@ -10,6 +10,5 @@
     <child link="shoot" />
   </joint>
-  <joint name="gimbal_joint" type="fixed">
-    <origin xyz="0 0 0" rpy="0 0 0" />
+  <joint name="gimbal_joint" type="floating">
     <parent link="odom" />
     <child link="gimbal_link" />
