Commit message: init

File: src/rm_gimbal_description/urdf/rm_gimbal_example.urdf.xacro (robot description, xacro)
@@ -26,3 +26,7 @@
     <child link="camera_optical_frame" />
   </joint>
+  <joint name="horizontal_camera_joint" type="floating">
+    <parent link="camera_optical_joint" />
+    <child link="horizontal_camera_joint" />
+  </joint>
 </robot>

Commit message: init

File: src/rm_gimbal_description/urdf/rm_gimbal_example.urdf.xacro (robot description, xacro)
@@ -26,7 +26,8 @@
     <child link="camera_optical_frame" />
   </joint>
+  <link name="horizontal_camera_link" />
   <joint name="horizontal_camera_joint" type="floating">
-    <parent link="camera_optical_joint" />
-    <child link="horizontal_camera_joint" />
+    <parent link="camera_optical_frame" />
+    <child link="horizontal_camera_link" />
   </joint>
 </robot>

Commit message: init

File: src/rm_gimbal_description/urdf/rm_gimbal_example.urdf.xacro (robot description, xacro)
@@ -7,5 +7,5 @@
   <joint name="shoot_joint" type="fixed">
     <origin xyz="0 0 0" rpy="0 0 0" />
-    <parent link="odom" />
+    <parent link="gimbal_link" />
     <child link="shoot" />
   </joint>
